Commit message: Imported upstream version '0.7.8' of 'upstream'

File: ign_ros2_control_demos/urdf/test_cart_effort.xacro.urdf (robot description, URDF)
Before this commit: robot cartopole, 3 links, 2 joints
Links:
- link cart: geometry visual box size=0.5 0.5 0.2
- link slideBar: geometry visual box size=30 0.05 0.05

File: ign_ros2_control_demos/urdf/test_cart_position.xacro.urdf (robot description, URDF)
Before this commit: robot cartopole, 3 links, 2 joints
Links:
- link cart: geometry visual box size=0.5 0.5 0.2
- link slideBar: geometry visual box size=30 0.05 0.05
