Commit message: Imported upstream version '1.2.7' of 'upstream'

File: gz_ros2_control_demos/urdf/test_cart_effort.xacro.urdf (robot description, URDF)
Before this commit: robot cartopole, 3 links, 2 joints
Links:
- link cart: geometry visual box size=0.5 0.5 0.2
- link slideBar: geometry visual box size=30 0.05 0.05
